Commit message: V10

File: simulation/models/urdf/humanoid.urdf (robot description, URDF)
Before this commit: robot humanoid_top_half, 16 links, 15 joints
Joints:
- joint left_shoulder_roll_joint: limit lower=-0.2618 upper=2.0944 effort=3.0 velocity=2.0944 -> lower=-0.8727 upper=2.0944 effort=3.0 velocity=2.0944
- joint right_shoulder_roll_joint: limit lower=-0.2618 upper=2.0944 effort=3.0 velocity=2.0944 -> lower=-0.8727 upper=2.0944 effort=3.0 velocity=2.0944

Commit message: trainging pick ad place

File: simulation/models/urdf/humanoid.urdf (robot description, URDF)
Before this commit: robot humanoid_top_half, 16 links, 15 joints
Links:
- link torso_link: geometry collision box size=0.09 0.07 0.30

Commit message: a

File: simulation/models/urdf/humanoid.urdf (robot description, URDF)
Before this commit: robot humanoid_top_half, 16 links, 15 joints
Links:
- added link left_shoulder_yaw_link; collision box size=0.025 0.025 0.025
- added link right_shoulder_yaw_link; collision box size=0.025 0.025 0.025
Joints:
- added joint left_shoulder_yaw_joint: type revolute, parent torso_link, child left_shoulder_yaw_link, origin xyz=0 0.11 0.05 rpy=0 0 0, axis 0 0 1, limit lower=-1.5708 upper=1.5708 effort=3.0 velocity=2.0944
- added joint right_shoulder_yaw_joint: type revolute, parent torso_link, child right_shoulder_yaw_link, origin xyz=0 -0.11 0.05 rpy=0 0 0, axis 0 0 1, limit lower=-1.5708 upper=1.5708 effort=3.0 velocity=2.0944
- joint left_shoulder_pitch_joint: origin xyz=0 0.11 0.05 rpy=0 0 0 -> xyz=0 0 0 rpy=0 0 0; parent torso_link -> left_shoulder_yaw_link
- joint right_shoulder_pitch_joint: origin xyz=0 -0.11 0.05 rpy=0 0 0 -> xyz=0 0 0 rpy=0 0 0; parent torso_link -> right_shoulder_yaw_link
